File: Noise Machine/Noise Machine.sch (KiCad schematic (older format))
At the start: 37 parts, among them Q1 2N2222A, Q2 2N3904, Q3 BC337, Q4 BC337, U1 LM386

Commit message: Add files via upload
Parts:
- added C10: 56p, symbol Device:C
- added D1, D2: 4148, symbol Device:D
- C13: renamed from C12; value 10u -> 10n
- C14: renamed from C13; value 10u -> 100n
- C15: renamed from C14; value 10u -> 10n
- C16: renamed from C15; value 10u -> 100n
- C9: value 56p -> 100n
- Q3, Q4: value BC337 -> BC547
- R10: value 1k -> 270
- R6: value 1k -> 10k
- renumbered C10 to C11, C11 to C12, D1 to D3, D2 to D4, D3 to D5, D4 to D6
Connections:
- net +5V: now also C9.1; no longer R7.1, R8.1
- net SQ_WAVE: now also C10.1, D2.2 (A); no longer C9.1
- net at C7.1, Q3.1 (C), R6.2: now also D1.2 (A)
- net at Q3.2 (B), R8.2: now also C10.2; no longer C9.2
- new net: C9.2, D1.1 (K), D2.1 (K), R7.1, R8.1
Other:
- moved on the sheet: R10, R6, R7, R8
