File: JAT EZ amp/JAT EZ amp.sch (KiCad schematic (older format))
At the start: 43 parts

Commit message: Add files via upload
Parts:
- gave numbers to parts that had none: 40
- renumbered CFB to CFB1, LL to LL1, RL to RL1

Commit message: Add files via upload
Parts:
- added CFB2: 100p, symbol Device:C
Connections:
- net GNDPWR: now also CFB2.1
- net at C7.1, L1.2, R15.1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: now also CFB2.2
Changed lines of the file:
@@
 Connection ~ 6000 1950
-Wire Wire Line
-	4850 2100 6500 2100
 Wire Wire Line
 	6500 2100 6500 2550
@@
 	0    1    1    0
 $EndComp
+$Comp
+L Device:C CFB2
+U 1 1 5F7EAA43
+P 6500 3850
+F 0 "CFB2" H 6385 3804 50  0000 R CNN
+F 1 "100p" H 6385 3895 50  0000 R CNN
+F 2 "" H 6538 3700 50  0001 C CNN
+F 3 "~" H 6500 3850 50  0001 C CNN
+	1    6500 3850
+	-1   0    0    1
+$EndComp
+$Comp
+L power:GNDS #PWR?
+U 1 1 5F7EB492
+P 6500 4050
+F 0 "#PWR?" H 6500 3800 50  0001 C CNN
+F 1 "GNDS" H 6505 3877 50  0000 C CNN
+F 2 "" H 6500 4050 50  0001 C CNN
+F 3 "" H 6500 4050 50  0001 C CNN
+	1    6500 4050
+	1    0    0    -1
+$EndComp
+Wire Wire Line
+	6500 4050 6500 4000
+Wire Wire Line
+	4850 2100 6500 2100
+Wire Wire Line
+	6500 3700 6500 3650
+Connection ~ 6500 3650
 $EndSCHEMATC

Commit message: Add files via upload
Connections:
- net GNDPWR: no longer CFB2.1
- net at CFB1.2, Q3.2 (B), R8.1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: now also CFB2.1
Other:
- moved on the sheet: CFB2, R8
Changed lines of the file:
@@
 L Device:R R8
 U 1 1 5F7D07B4
-P 4850 3400
-F 0 "R8" H 4780 3354 50  0000 R CNN
-F 1 "22k" H 4780 3445 50  0000 R CNN
-F 2 "" V 4780 3400 50  0001 C CNN
-F 3 "~" H 4850 3400 50  0001 C CNN
-	1    4850 3400
-	-1   0    0    1
+P 5400 2100
+F 0 "R8" H 5330 2054 50  0000 R CNN
+F 1 "22k" H 5330 2145 50  0000 R CNN
+F 2 "" V 5330 2100 50  0001 C CNN
+F 3 "~" H 5400 2100 50  0001 C CNN
+	1    5400 2100
+	0    -1   -1   0
 $EndComp
 $Comp
@@
 	3650 3950 3650 4050
 Wire Wire Line
-	4850 3650 4850 3550
-Wire Wire Line
 	4850 3650 4850 3750
-Connection ~ 4850 3650
 Wire Wire Line
 	4850 4050 4850 4150
@@
 Wire Wire Line
 	4400 3650 4450 3650
-Wire Wire Line
-	4850 2100 4850 3250
 $Comp
 L Device:C CFB1
@@
 L Device:C CFB2
 U 1 1 5F7EAA43
-P 6500 3850
-F 0 "CFB2" H 6385 3804 50  0000 R CNN
-F 1 "100p" H 6385 3895 50  0000 R CNN
-F 2 "" H 6538 3700 50  0001 C CNN
-F 3 "~" H 6500 3850 50  0001 C CNN
-	1    6500 3850
-	-1   0    0    1
-$EndComp
-$Comp
-L power:GNDS #PWR?
-U 1 1 5F7EB492
-P 6500 4050
-F 0 "#PWR?" H 6500 3800 50  0001 C CNN
-F 1 "GNDS" H 6505 3877 50  0000 C CNN
-F 2 "" H 6500 4050 50  0001 C CNN
-F 3 "" H 6500 4050 50  0001 C CNN
-	1    6500 4050
-	1    0    0    -1
-$EndComp
-Wire Wire Line
-	6500 4050 6500 4000
-Wire Wire Line
-	4850 2100 6500 2100
-Wire Wire Line
-	6500 3700 6500 3650
-Connection ~ 6500 3650
+P 5400 2550
+F 0 "CFB2" H 5285 2504 50  0000 R CNN
+F 1 "100p" H 5285 2595 50  0000 R CNN
+F 2 "" H 5438 2400 50  0001 C CNN
+F 3 "~" H 5400 2550 50  0001 C CNN
+	1    5400 2550
+	0    -1   -1   0
+$EndComp
+Wire Wire Line
+	6500 2100 5700 2100
+Wire Wire Line
+	5700 2100 5700 2550
+Wire Wire Line
+	5700 2550 5550 2550
+Connection ~ 5700 2100
+Wire Wire Line
+	5700 2100 5550 2100
+Wire Wire Line
+	5250 2100 4850 2100
+Wire Wire Line
+	4850 2100 4850 2550
+Connection ~ 4850 3650
+Wire Wire Line
+	4850 2550 5250 2550
+Connection ~ 4850 2550
+Wire Wire Line
+	4850 2550 4850 3650
 $EndSCHEMATC
