File: Power Supplies/eevblog power supply/psu.sch (KiCad schematic (older format))
At the start: 28 parts, among them Q1 3904, U1 TL431LP, U2 LM324, U3 LM1117

Commit message: Add files via upload
Parts:
- added BT1: Battery, symbol Device:Battery
- added C5, C6: 100n, symbol Device:C_Small
- added D2: OC_LED, symbol Device:LED
- added D3: PWR_LED, symbol Device:LED
- added OC_THRES1: 5k, symbol Device:R_POT_TRIM_US
- added Q2, Q3: 2n7000, symbol Device:Q_NMOS_SGD
- added Q4: IRLZ44N, Package_TO_SOT_THT:TO-220-3_Vertical, symbol Transistor_FET:IRLZ44N
- added R16: 27k, symbol Device:R_US
- added R17: 5.1k, symbol Device:R_US
- added R18, R22, R24: 1k, symbol Device:R_US
- added R19, R20: 10k, symbol Device:R_US
- added R21: 100k, symbol Device:R_US
- added R23: 2.7k, symbol Device:R_US
- added SW1: RESET, symbol Switch:SW_DIP_x01
- added SW2: SW_SPST, symbol Switch:SW_SPST
- added U4: LM358, symbol Amplifier_Operational:LM358
- R2: value 15k -> 27k
Connections:
- net labels added: +BATT, LOAD_Hi, LOAD_Lo
- net labels removed: +12V, V_OUT
- wire segments 81 -> 143
Other:
- moved on the sheet: C1, C4, D1, R1, R13, R15, U1, U2E
