File: Noise Machine V1.1/Noise Machine.sch (KiCad schematic (older format))
At the start: 49 parts, among them Q1 2N2222A, Q1 2n2222, Q2 2N3904, Q2 2n2222, Q3 2n2907, Q3 S8050, Q4 S8050

Commit message: Re-organize structure
Parts:
- removed C3: 100u, Capacitor_THT:CP_Radial_D6.3mm_P2.50mm, symbol Device:CP1
- removed C5: 470u, Capacitor_THT:CP_Radial_D8.0mm_P2.50mm, symbol Device:CP1
- removed C6, C?: 1u, symbol Device:C
- removed D1, D2: 1n4007, Diode_THT:D_DO-41_SOD81_P7.62mm_Horizontal, symbol Device:D
- removed L?: 1mH, symbol Device:L
- removed LS1: 8R, symbol Device:Speaker
- removed Q1, Q2: 2n2222, Package_TO_SOT_THT:TO-92, symbol Device:Q_NPN_EBC
- removed Q3: 2n2907, Package_TO_SOT_THT:TO-92, symbol Device:Q_PNP_EBC
- removed R3: 4.7k, Resistor_THT:R_Axial_DIN0207_L6.3mm_D2.5mm_P7.62mm_Horizontal, symbol Device:R_US
- removed R4, R5: 470, Resistor_THT:R_Axial_DIN0207_L6.3mm_D2.5mm_P7.62mm_Horizontal, symbol Device:R_US
- removed R6, R7: .47, Resistor_THT:R_Axial_DIN0207_L6.3mm_D2.5mm_P7.62mm_Horizontal, symbol Device:R_US
- removed RV1: 10k, Potentiometer_THT:Potentiometer_ACP_CA9-H5_Horizontal, symbol Device:R_POT_US
- removed RV2: 20k, Potentiometer_THT:Potentiometer_ACP_CA9-H5_Horizontal, symbol Device:R_POT_TRIM_US
- added C? (x3): 10u, symbol Device:C
- added C?: 22n, symbol Device:C
- added C?: 470u, Capacitor_THT:CP_Radial_D8.0mm_P2.50mm, symbol Device:CP1
- added D? (x2): 1n4007, Diode_THT:D_DO-41_SOD81_P7.62mm_Horizontal, symbol Device:D
- added LS?: 8R, symbol Device:Speaker
- added Q? (x2): 2N2222, Package_TO_SOT_THT:TO-92, symbol Device:Q_NPN_EBC
- added Q?: 2n2907, symbol Device:Q_PNP_ECB
- added Q?: 2n2222, symbol Device:Q_NPN_ECB
- added R? (x2): 1k, symbol Device:R_US
- added R?: 100k, symbol Device:R_US
- added R?: 51k, symbol Device:R_US
- added R?: 510, symbol Device:R_US
- added R? (x2): 27k, symbol Device:R_US
- added R? (x2): .47, Resistor_THT:R_Axial_DIN0207_L6.3mm_D2.5mm_P7.62mm_Horizontal, symbol Device:R_US
- added RV?: 10k, symbol Device:R_POT_US
- C14: renamed from C15; value 1u -> 10u
- C3: value 100p -> 10n
- C4: value 22n -> 2.2n
- Q2: value 2N3904 -> 2N2222
- Q3: value S8050 -> 2N2222
- Q7: renamed from Q4; value S8050 -> 2N2222
- gave numbers to parts that had none: 4
- renumbered C13 to C12, C14 to C13, C5 to C6, C7 to C8, R3 to R1, R7 to R11, R8 to R14, R10 to R17, R1 to R2, R2 to R3, R5 to R6, R4 to R8, R6 to R9
Connections:
- net labels added: SIG_COLOR, ~Q
- net labels removed: Q!, SIG_OUT
- wire segments 113 -> 130
Other:
- note removed: "Hi pass"
- note removed: "Lo pass"
- note removed: "With these components and values, I get a noise signal at about 1Vpp. \nThis will be attenuated significantly in the filter stage, \nbut gain can be adjusted somewhat by increasing R4"
- moved on the sheet: C1, C10, C12, C13, C14, C2, C3, C4, C5, C6, C8, D3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

Commit message: add new circuits
Parts:
- removed C5: 1u, symbol Device:C
- removed C? (x3): 10u, symbol Device:C
- removed C?: 22n, symbol Device:C
- removed C?: 470u, Capacitor_THT:CP_Radial_D8.0mm_P2.50mm, symbol Device:CP1
- removed D? (x2): 1n4007, Diode_THT:D_DO-41_SOD81_P7.62mm_Horizontal, symbol Device:D
- removed Q? (x2): 2N2222, Package_TO_SOT_THT:TO-92, symbol Device:Q_NPN_EBC
- removed Q?: 2n2907, symbol Device:Q_PNP_ECB
- removed Q?: 2n2222, symbol Device:Q_NPN_ECB
- removed R4, R? (x2): 27k, symbol Device:R_US
- removed R7: 270, symbol Device:R_US
- removed R8, R? (x2): 1k, symbol Device:R_US
- removed R?: 100k, symbol Device:R_US
- removed R?: 51k, symbol Device:R_US
- removed R?: 510, symbol Device:R_US
- removed R? (x2): .47, Resistor_THT:R_Axial_DIN0207_L6.3mm_D2.5mm_P7.62mm_Horizontal, symbol Device:R_US
- removed RV?: 10k, symbol Device:R_POT_US
- added C11, C12, C13: 1u, Capacitor_SMD:C_0603_1608Metric_Pad1.08x0.95mm_HandSolder, symbol Device:C
- added J1: PWR, Connector_PinHeader_2.54mm:PinHeader_1x02_P2.54mm_Vertical, symbol Connector:Conn_01x02_Male
- added RV2: 20k, Connector_PinHeader_2.54mm:PinHeader_1x02_P2.54mm_Vertical, symbol Device:R_POT_US
- added Ri1: 5.1k, Resistor_SMD:R_0603_1608Metric_Pad0.98x0.95mm_HandSolder, symbol Device:R_US
- added U1: NS8002, Package_SO:SO-8_3.9x4.9mm_P1.27mm, symbol 8002:8002_Small
- C1: footprint (none) -> Capacitor_SMD:C_0603_1608Metric_Pad1.08x0.95mm_HandSolder
- C10: renamed from C4; value 2.2n -> 22n; footprint (none) -> Capacitor_SMD:C_0603_1608Metric_Pad1.08x0.95mm_HandSolder
- C2: renamed from C3; value 10n -> 1n; footprint (none) -> Capacitor_SMD:C_0603_1608Metric_Pad1.08x0.95mm_HandSolder
- C3: renamed from C8; footprint (none) -> Capacitor_SMD:C_0603_1608Metric_Pad1.08x0.95mm_HandSolder
- C4: renamed from C6; footprint (none) -> Capacitor_SMD:C_0603_1608Metric_Pad1.08x0.95mm_HandSolder
- C5: renamed from C10; footprint (none) -> Capacitor_SMD:C_0603_1608Metric_Pad1.08x0.95mm_HandSolder
- C6: renamed from C12; footprint (none) -> Capacitor_SMD:C_0603_1608Metric_Pad1.08x0.95mm_HandSolder
- C7: renamed from C13; footprint (none) -> Capacitor_SMD:C_0603_1608Metric_Pad1.08x0.95mm_HandSolder
- C8: renamed from C2; footprint (none) -> Capacitor_SMD:C_0603_1608Metric_Pad1.08x0.95mm_HandSolder
- C9: renamed from C14; footprint (none) -> Capacitor_SMD:C_0603_1608Metric_Pad1.08x0.95mm_HandSolder
- D1: renamed from D3; footprint (none) -> Diode_THT:D_DO-35_SOD27_P5.08mm_Vertical_AnodeUp
- D2: renamed from D4; footprint (none) -> Diode_THT:D_DO-35_SOD27_P5.08mm_Vertical_AnodeUp
- D3: renamed from D5; footprint (none) -> Diode_THT:D_DO-35_SOD27_P5.08mm_Vertical_AnodeUp
- LS1: renamed from LS?; value 8R -> 3R-8R; footprint (none) -> Connector_PinHeader_2.54mm:PinHeader_1x02_P2.54mm_Vertical
- Q1, Q2: footprint (none) -> Package_TO_SOT_SMD:SOT-23; symbol Device:Q_NPN_EBC -> Device:Q_NPN_BEC
- Q3: footprint (none) -> Package_TO_SOT_SMD:SOT-23; symbol Device:Q_NPN_CBE -> Device:Q_NPN_BEC
- Q4: renamed from Q7; footprint (none) -> Package_TO_SOT_SMD:SOT-23; symbol Device:Q_NPN_CBE -> Device:Q_NPN_BEC
- R1: footprint (none) -> Resistor_SMD:R_0603_1608Metric_Pad0.98x0.95mm_HandSolder
- R2: renamed from R9; footprint (none) -> Resistor_SMD:R_0603_1608Metric_Pad0.98x0.95mm_HandSolder
- R3: renamed from R5; footprint (none) -> Resistor_SMD:R_0603_1608Metric_Pad0.98x0.95mm_HandSolder
- R4: renamed from R11; footprint (none) -> Resistor_SMD:R_0603_1608Metric_Pad0.98x0.95mm_HandSolder
- R5: renamed from R14; footprint (none) -> Resistor_SMD:R_0603_1608Metric_Pad0.98x0.95mm_HandSolder
- R6: renamed from R17; footprint (none) -> Resistor_SMD:R_0603_1608Metric_Pad0.98x0.95mm_HandSolder
- R7: renamed from R2; footprint (none) -> Resistor_SMD:R_0603_1608Metric_Pad0.98x0.95mm_HandSolder
- R8: renamed from R3; footprint (none) -> Resistor_SMD:R_0603_1608Metric_Pad0.98x0.95mm_HandSolder
- R9: renamed from R6; footprint (none) -> Resistor_SMD:R_0603_1608Metric_Pad0.98x0.95mm_HandSolder
- RV1: footprint (none) -> Connector_PinHeader_2.54mm:PinHeader_1x03_P2.54mm_Vertical
Connections:
- net labels removed: Q, SIG_COLOR, SIG_NOISE, ~Q
- wire segments 130 -> 101
Other:
- note added: "Av=2(RV2/Ri)"
- moved on the sheet: C1, C10, C2, C4, C6, C8, D1, D2, D3, LS1, Q1, Q2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
